File: adc.sch (EAGLE design)
At the start: 1 part, among them U1 ADV7173KSTZ

Commit message: placa ADC v1
Parts:
- added C1, C10, C12, C3, C5, C6, C7, C8, C9: 10nf, eagle-ltspice:CC0603
- added C11, C13, C2, C4: 10uf, eagle-ltspice:CC0603
- added D1, D2, D3, D4, D5, D6: PMLL4150, diode:PMLL4150
- added IC13, IC5, IC6: 4051D, 40xx:4051D
- added JP1, JP2, JP3: (no value), jumper:JP2E
- added R1, R10, R11, R12, R13, R14, R15, R16, R17, R18, R19, R2, R20, R21, R22, R23, R24, R25, R26, R27, R28, R29, R3, R30, R31, R32, R33, R34, R35, R36, R37, R38, R39, R4, R40, R41, R42, R43, R44, R45, R46, R47, R5, R6, R7, R8, R9: (no value), SparkFun:RESISTOR0603
- added SV1, SV2: (no value), con-lstb:MA20-2
- added U$1, U$2: POT100K_3362U, SparkFun:POT100K_3362U
- added U2, U5, U6, U7: AD5308ARUZ, Analog Devices_By_element14_Batch_1:AD5308ARUZ
- added U3: AD7927BRUZ, Analog Devices_By_element14_Batch_1:AD7927BRUZ
- added U4: ADV7173KSTZ, ADI-Phase-2:ADV7173KSTZ
Connections:
- new net +2,5V_ADCREF: U1.VREF_A, U1.VREF_B, U4.VREF_A, U4.VREF_B
- new net CH_A(ADC): D1.A, D2.C, R17.1, U1.+INA, U5.OUTC
- new net CH_B(ADC): D3.A, D4.C, R33.1, U4.+IN_B, U6.OUTC
- new net CH_C(ADC): D5.A, D6.C, R47.1, U4.+INA, U7.OUTC
- new net DAC_OUT: R1.2, U$1.A, U2.OUTA
- new net DCLK: U1.CLK_A, U1.CLK_B, U4.CLK_A, U4.CLK_B
- new net DFS/GAIN: JP1.2, U1.DFS_GAIN, U4.DFS_GAIN
- new net DGND: C12.2, C13.2, C3.2, C4.2, C5.2, JP1.3, JP2.3, JP3.3, U1.GND, U1.GND_(, U1.GND_10, U1.GND_11, U1.GND_12, U1.GND_7, U1.GND_8, U1.GND_9, U3.GND, U3.IOUT2, U3.R/W, U3.RFB, U4.GND, U4.GND_(, U4.GND_10, U4.GND_11, U4.GND_12, U4.GND_7, U4.GND_8, U4.GND_9
- new net GND: C1.2, C10.2, C11.2, C2.2, C7.2, C9.2, D2.A, D4.A, D6.A, R19.2, R22.2, R32.2, R36.2, R46.2, R8.2, U1.-INA, U2.+IND, U4.-INA
- new net N$1: C7.1, R2.1, U2.+INB
- new net N$10: SV2.29, U1.D5_A
- new net N$100: U5.-INA, U5.OUTA
- new net N$101: R31.1, R32.1, U6.-INC
- new net N$102: R37.2, R38.2, R39.2, R40.2, R41.2, R42.2, R43.2, R44.2
- new net N$103: U6.-INA, U6.OUTA
- new net N$104: R45.1, R46.1, U7.-INC
- new net N$105: U7.-INA, U7.OUTA
- new net N$106: R35.1, U7.+INA
- new net N$107: R21.1, U6.+INA
- new net N$109: R20.2, R21.2, R34.2, R35.2, R6.2, R7.2, U$2.A, U2.OUTD
- new net N$11: SV2.40, U1.D0_B
- new net N$12: SV2.30, U1.D5_B
- new net N$13: SV2.32, U1.D4_B
- new net N$14: SV2.39, U1.D0_A
- new net N$15: SV2.31, U1.D4_A
- new net N$16: SV2.25, U1.D7_A
- new net N$17: SV2.34, U1.D3_B
- new net N$18: SV2.27, U1.D6_A
- new net N$19: SV2.35, U1.D2_A
- new net N$2: C6.1, R1.1, R2.2
- new net N$20: SV2.37, U1.D1_A
- new net N$21: SV2.36, U1.D2_B
- new net N$22: SV2.28, U1.D6_B
- new net N$23: SV2.26, U1.D7_B(MSB)
- new net N$24: SV2.2, U3.DB11
- new net N$25: SV2.38, U1.D1_B
- new net N$26: SV2.4, U3.DB10
- new net N$27: SV2.6, U3.DB9
- new net N$28: SV2.8, U3.DB8
- new net N$29: SV2.10, U3.DB7
- new net N$3: C5.1, U$1.E, U$1.S, U2.-INA, U3.IOUT1
- new net N$30: SV2.12, U3.DB6
- new net N$31: SV2.14, U3.DB5
- new net N$32: SV2.16, U3.DB4
- new net N$33: SV2.18, U3.DB3
- new net N$34: SV2.20, U3.DB2
- new net N$35: SV2.22, U3.DB1
- new net N$36: SV2.24, U3.DB0(LSB)
- new net N$37: SV2.1, U3.CS
- new net N$38: IC5A.X0, R9.1
- new net N$39: IC5A.X1, R10.1
- new net N$4: C6.2, R3.2, U2.-INB, U2.OUTB
- new net N$40: IC5A.X2, R11.1
- new net N$41: IC5A.X4, R12.1
- new net N$42: IC5A.X3, R13.1
- new net N$43: IC5A.X5, R14.1
- new net N$44: IC5A.X6, R15.1
- new net N$45: IC5A.X7, R16.1
- new net N$46: IC6A.X0, R23.1
- new net N$47: IC6A.X1, R24.1
- new net N$48: R23.2, R24.2, R25.2, R26.2, R27.2, R28.2, R29.2, R30.2
- new net N$49: R10.2, R11.2, R12.2, R13.2, R14.2, R15.2, R16.2, R9.2
- new net N$5: C9.1, R4.1, U2.+INC
- new net N$50: R18.1, R19.1, U5.-INC
- new net N$51: IC5A.X, R17.2, U5.+INC
- new net N$52: IC6A.X2, R25.1
- new net N$53: IC6A.X4, R26.1
- new net N$54: IC6A.X3, R27.1
- new net N$55: IC6A.X5, R28.1
- new net N$56: IC6A.X6, R29.1
- new net N$57: IC6A.X7, R30.1
- new net N$58: R31.2, U6.-INB, U6.OUTB
- new net N$59: R45.2, U7.-INB, U7.OUTB
- new net N$6: C8.1, R3.1, R4.2
- new net N$60: IC13A.X, R47.2, U7.+INC
- new net N$61: IC6A.X, R33.2, U6.+INC
- new net N$62: IC13A.X0, R37.1
- new net N$63: IC13A.X1, R38.1
- new net N$64: IC13A.X2, R39.1
- new net N$65: IC13A.X4, R40.1
- new net N$66: IC13A.X3, R41.1
- new net N$67: IC13A.X5, R42.1
- new net N$68: IC13A.X6, R43.1
- new net N$69: IC13A.X7, R44.1
- new net N$7: C8.2, R5.2, U2.-INC, U2.OUTC
- new net N$70: R34.1, R36.1, U7.+INB
- new net N$71: R6.1, R8.1, U5.+INB
- new net N$72: R20.1, R22.1, U6.+INB
- new net N$73: R7.1, U5.+INA
- new net N$74: SV1.33, U4.D3_A
- new net N$75: SV1.29, U4.D5_A
- new net N$76: SV1.40, U4.D0_B
- new net N$77: SV1.30, U4.D5_B
- new net N$78: SV1.32, U4.D4_B
- new net N$79: SV1.39, U4.D0_A
- new net N$8: R5.1, U$2.E, U$2.S, U2.-IND
- new net N$80: SV1.31, U4.D4_A
- new net N$81: SV1.25, U4.D7_A
- new net N$82: SV1.34, U4.D3_B
- new net N$83: SV1.27, U4.D6_A
- new net N$84: SV1.35, U4.D2_A
- new net N$85: SV1.37, U4.D1_A
- new net N$86: SV1.36, U4.D2_B
- new net N$87: SV1.28, U4.D6_B
- new net N$88: SV1.26, U4.D7_B(MSB)
- new net N$89: SV1.38, U4.D1_B
- new net N$9: SV2.33, U1.D3_A
- new net N$90: IC5A.C, SV2.3
- new net N$91: IC5A.B, SV2.5
- new net N$92: IC5A.A, SV2.7
- new net N$93: IC13A.C, SV1.1
- new net N$94: IC13A.B, SV1.3
- new net N$95: IC13A.A, SV1.5
- new net N$96: IC6A.C, SV1.7
- new net N$97: IC6A.B, SV1.9
- new net N$98: IC6A.A, SV1.11
- new net N$99: R18.2, U5.-INB, U5.OUTB
- new net S1: JP2.2, U1.S1, U4.S1
- new net S2: JP3.2, U1.S2, U4.S2
- new net VCC: C1.1, C10.1, C11.1, C2.1, D1.C, D3.C, D5.C, IC13A.INH, IC5A.INH, IC6A.INH, U1.VD1, U1.VD2, U1.VD3, U1.VD4, U4.VD2, U4.VD3, U4.VD4
- new net VDD: C12.1, C13.1, C3.1, C4.1, JP1.1, JP2.1, JP3.1, U1.VDD1, U1.VDD2, U1.VDD4, U1.VDD6, U2.V+, U2.V-, U3.VDD, U3.VREF, U4.VDD1, U4.VDD2, U4.VDD4, U4.VDD6, U5.V+, U5.V-, U6.V+, U6.V-, U7.V+, U7.V-
Other:
- moved on the sheet: U1

Commit message: VHDL
Parts:
- removed D1, D2, D3, D4, D5, D6: PMLL4150, diode:PMLL4150
Connections:
- removed net N$85: SV1.37, U4.D1_A
- removed net N$92: IC5A.A, SV2.7
- new net +5V: SV1.30, SV2.30, U2.V+, U5.V+, U6.V+, U7.V+
- new net -5V: U2.V-, U5.V-, U6.V-, U7.V-
- new net N$110: IC5A.A, SV2.20
- new net N$111: SV2.16, U3.CS
- net CH_A(ADC): no longer D1.A, D2.C
- net CH_B(ADC): no longer D3.A, D4.C
- net CH_C(ADC): no longer D5.A, D6.C
- net DGND: now also SV1.11, SV1.12, SV2.11, SV2.12
- net GND: no longer D2.A, D4.A, D6.A
- net N$10: now also SV2.25; no longer SV2.29
- net N$11: now also SV2.39; no longer SV2.40
- net N$12: now also SV2.32; no longer SV2.30
- net N$13: now also SV2.34; no longer SV2.32
- net N$14: now also SV2.37; no longer SV2.39
- net N$15: now also SV2.27; no longer SV2.31
- net N$16: now also SV2.21; no longer SV2.25
- net N$17: now also SV2.36; no longer SV2.34
- net N$18: now also SV2.23; no longer SV2.27
- net N$19: now also SV2.33; no longer SV2.35
- net N$20: now also SV2.35; no longer SV2.37
- net N$21: now also SV2.38; no longer SV2.36
- net N$24: now also SV2.13; no longer SV2.2
- net N$25: now also SV2.40; no longer SV2.38
- net N$26: now also SV2.9; no longer SV2.4
- net N$27: now also SV2.7; no longer SV2.6
- net N$28: now also SV2.5; no longer SV2.8
- net N$29: now also SV2.3; no longer SV2.10
- net N$30: now also SV2.1; no longer SV2.12
- net N$31: now also SV2.2; no longer SV2.14
- net N$32: now also SV2.4; no longer SV2.16
- net N$33: now also SV2.6; no longer SV2.18
- net N$34: now also SV2.8; no longer SV2.20
- net N$35: now also SV2.10; no longer SV2.22
- net N$36: now also SV2.14; no longer SV2.24
- net N$37: now also SV1.38, U4.D0_A; no longer SV2.1, U3.CS
- net N$74: now also SV1.40, U4.D1_A; no longer SV1.33, U4.D3_A
- net N$75: now also SV1.39, U4.D2_A; no longer SV1.29, U4.D5_A
- net N$76: now also SV1.36; no longer SV1.40
- net N$77: now also SV1.24; no longer SV1.30
- net N$78: now also SV1.26; no longer SV1.32
- net N$79: now also SV1.37, U4.D3_A; no longer SV1.39, U4.D0_A
- net N$80: now also SV1.35; no longer SV1.31
- net N$81: now also SV1.33, U4.D5_A; no longer SV1.25, U4.D7_A
- net N$82: now also SV1.28; no longer SV1.34
- net N$83: now also SV1.31; no longer SV1.27
- net N$84: now also SV1.27, U4.D7_A; no longer SV1.35, U4.D2_A
- net N$86: now also SV1.32; no longer SV1.36
- net N$87: now also SV1.22; no longer SV1.28
- net N$88: now also SV1.20; no longer SV1.26
- net N$89: now also SV1.34; no longer SV1.38
- net N$9: now also SV2.31; no longer SV2.33
- net N$90: now also SV2.24; no longer SV2.3
- net N$91: now also SV2.22; no longer SV2.5
- net N$93: now also SV1.19; no longer SV1.1
- net N$94: now also SV1.15; no longer SV1.3
- net N$95: now also SV1.13; no longer SV1.5
- net N$96: now also SV1.25; no longer SV1.7
- net N$97: now also SV1.23; no longer SV1.9
- net N$98: now also SV1.21; no longer SV1.11
- net VCC: no longer D1.C, D3.C, D5.C
- net VDD: now also SV1.29, SV2.29; no longer U2.V+, U2.V-, U5.V+, U5.V-, U6.V+, U6.V-, U7.V+, U7.V-

Commit message: autalização
Parts:
- added X1: (no value), con-ptr500:AK300/5
Connections:
- removed net DGND: C12.2, C13.2, C3.2, C4.2, C5.2, JP1.3, JP2.3, JP3.3, SV1.11, SV1.12, SV2.11, SV2.12, U1.GND, U1.GND_(, U1.GND_10, U1.GND_11, U1.GND_12, U1.GND_7, U1.GND_8, U1.GND_9, U3.GND, U3.IOUT2, U3.R/W, U3.RFB, U4.GND, U4.GND_(, U4.GND_10, U4.GND_11, U4.GND_12, U4.GND_7, U4.GND_8, U4.GND_9
- net +2,5V_ADCREF: now also X1-3.KL
- net +5V: now also X1-5.KL
- net -5V: now also X1-4.KL
- net DCLK: now also SV1.10
- net GND: now also C12.2, C13.2, C3.2, C4.2, C5.2, JP1.3, JP2.3, JP3.3, SV1.11, SV1.29, SV2.11, SV2.29, U1.GND, U1.GND_(, U1.GND_10, U1.GND_11, U1.GND_12, U1.GND_7, U1.GND_8, U1.GND_9, U3.GND, U3.IOUT2, U3.R/W, U3.RFB, U4.GND, U4.GND_10, U4.GND_11, U4.GND_12, U4.GND_7, U4.GND_8, U4.GND_9, X1-1.KL
- net N$93: now also SV1.17; no longer SV1.19
- net VDD: now also SV1.12, SV2.12, X1-2.KL; no longer SV1.29, SV2.29

Commit message: Atualização
VHDL com SWITCH CASE. 1-16 start end package
C# com controle de erro
ADC com alterações
Parts:
- removed X1: (no value), con-ptr500:AK300/5
- added X2: (no value), con-ptr500:AK300/6
Connections:
- removed net N$100: U5.-INA, U5.OUTA
- removed net N$103: U6.-INA, U6.OUTA
- removed net N$105: U7.-INA, U7.OUTA
- new net 1V: U3.VREF, X2-2.KL
- net +2,5V_ADCREF: now also X2-3.KL; no longer X1-3.KL
- net +5V: now also SV1.12, SV2.12, X2-5.KL; no longer SV1.30, SV2.30, X1-5.KL
- net -5V: now also X2-4.KL; no longer X1-4.KL
- net GND: now also X2-1.KL; no longer X1-1.KL
- net N$102: now also U7.-INA, U7.OUTA
- net N$110: now also SV2.15; no longer SV2.20
- net N$48: now also U6.-INA, U6.OUTA
- net N$49: now also U5.-INA, U5.OUTA
- net N$90: now also SV2.19; no longer SV2.24
- net N$91: now also SV2.17; no longer SV2.22
- net VCC: now also U4.VD1
- net VDD: now also SV1.30, SV2.30, X2-6.KL; no longer SV1.12, SV2.12, U3.VREF, X1-2.KL

Commit message: ADC update
Atualizado algumas trilhas e GND não conectado
Parts:
- removed R47: (no value), SparkFun:RESISTOR0603
- removed U$2: POT100K_3362U, SparkFun:POT100K_3362U
- added R48, R49, R50, R51, R52, R53, R54, R55, R56, R57: (no value), SparkFun:RESISTOR0603
Connections:
- removed net N$109: R20.2, R21.2, R34.2, R35.2, R6.2, R7.2, U$2.A, U2.OUTD
- removed net N$59: R45.2, U7.-INB, U7.OUTB
- new net N$103: C5.1, R48.2, U3.IOUT1
- new net N$105: R18.2, R5.1, U5.OUTA
- new net N$114: R55.2, R56.1, U7.-INC
- new net N$117: R51.2, R53.1, U5.-INC
- new net N$119: R55.1, R57.2, U7.OUTB
- new net N$120: R17.1, R31.2, U6.OUTA
- new net N$121: R50.2, R52.1, U6.OUTB
- new net N$122: IC6A.X, R50.1, U6.-INB
- net CH_A(ADC): now also R53.2; no longer R17.1
- net CH_B(ADC): now also R54.2; no longer R33.1
- net CH_C(ADC): now also R56.2; no longer R47.1
- net GND: now also U1.-IN_B, U1.VREF_OUT, U4.-IN_B, U4.GND_(, U4.VREF_OUT; no longer U2.+IND
- net N$101: now also U6.+INC; no longer U6.-INC
- net N$102: now also R33.2; no longer U7.OUTA
- net N$104: now also U7.+INC; no longer U7.-INC
- net N$3: now also R48.1; no longer C5.1, U3.IOUT1
- net N$48: now also R17.2; no longer U6.OUTA
- net N$49: now also R5.2; no longer U5.OUTA
- net N$50: now also U5.+INC; no longer U5.-INC
- net N$51: now also R49.2, R51.1, U5.OUTB; no longer IC5A.X, R17.2, U5.+INC
- net N$58: now also R52.2, R54.1, U6.-INC; no longer R31.2, U6.-INB, U6.OUTB
- net N$60: now also R33.1, R45.2, U7.OUTA; no longer IC13A.X, R47.2, U7.+INC
- net N$61: now also IC13A.X, R57.1, U7.-INB; no longer IC6A.X, R33.2, U6.+INC
- net N$7: now also R20.2, R21.2, R34.2, R35.2, R6.2, R7.2; no longer R5.2
- net N$8: now also U2.+IND; no longer R5.1, U$2.E, U$2.S, U2.-IND
- net N$99: now also IC5A.X, R49.1; no longer R18.2, U5.OUTB
Other:
- moved on the sheet: R17, R33, R5
